Commit message: bug: fixed laser frame_id in urdf

File: osracer_description/urdf/osracer.urdf (robot description, URDF)
Before this commit: robot osracer, 11 links, 10 joints
Links:
- removed link laser_link
- added link laser, mass 0.160; collision mesh filename=package://osracer_description/meshes/laser.STL; visual mesh filename=package://osracer_description/meshes/laser.STL
Joints:
- joint laser_joint: child laser_link -> laser

Commit message: bug: fixed the prim path of laser_link in urdf

File: osracer_description/urdf/osracer.urdf (robot description, URDF)
Before this commit: robot osracer, 11 links, 10 joints
Links:
- link laser: geometry collision mesh filename=package://osracer_description/meshes/laser_link.STL; visual mesh filename=package://osracer_description/meshes/laser_link.STL

Commit message: fix(urdf): zero laser_joint roll/pitch for gmapping planar scan

File: osracer_description/urdf/osracer.urdf (robot description, URDF)
Before this commit: robot osracer, 11 links, 10 joints
Joints:
- joint laser_joint: origin xyz=-0.082558 -0.017229 0.034095 rpy=-0.00028339 -0.031729 0.0057633 -> xyz=-0.082558 -0.017229 0.034095 rpy=0 0 0

Commit message: fix: align navigation parameters with ackermann chassis

File: osracer_description/urdf/osracer.urdf (robot description, URDF)
Before this commit: robot osracer, 11 links, 10 joints
Joints:
- joint left_steering_hinge_joint: limit (none) -> lower=-0.5236 upper=0.5236 effort=5 velocity=2.0; type continuous -> revolute
- joint right_steering_hinge_joint: limit (none) -> lower=-0.5236 upper=0.5236 effort=5 velocity=2.0; type continuous -> revolute
