Commit message: refactor: streamline public runtime ownership

File: osracer_description/urdf/osracer.urdf (robot description, URDF)
Before this commit: robot osracer, 11 links, 10 joints
Links:
- link Left_front_wheel_link: geometry collision mesh filename=package://osracer_description/meshes/Left_front_wheel_link.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 scale=0.941 1 0.941; visual mesh filename=package://osracer_description/meshes/Left_front_wheel_link.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 scale=0.941 1 0.941
- link left_rear_wheel_link: geometry collision mesh filename=package://osracer_description/meshes/left_rear_wheel_link.S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 scale=0.941 1 0.941; visual mesh filename=package://osracer_description/meshes/left_rear_wheel_link.S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 scale=0.941 1 0.941
- link right_front_wheel_link: geometry collision mesh filename=package://osracer_description/meshes/right_front_wheel_link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 scale=0.941 1 0.941; visual mesh filename=package://osracer_description/meshes/right_front_wheel_link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 scale=0.941 1 0.941
- link right_rear_wheel_link: geometry collision mesh filename=package://osracer_description/meshes/right_rear_wheel_link.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 scale=0.941 1 0.941; visual mesh filename=package://osracer_description/meshes/right_rear_wheel_link.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 scale=0.941 1 0.941
Joints:
- joint left_rear_wheel_joint: origin xyz=-0.18068 0.10027 -0.10041 rpy=0 0 0 -> xyz=-0.17785021060022 0.09027 -0.10041 rpy=0 0 0
- joint left_steering_hinge_joint: origin xyz=0.11108 0.088168 -0.10247 rpy=0 0 0 -> xyz=0.11108 0.078168 -0.10247 rpy=0 0 0
- joint right_rear_wheel_joint: origin xyz=-0.180681048799559 -0.134728618898254 -0.100407328161273 rpy=0 0 0 -> xyz=-0.177851259399779 -0.124728618898254 -0.100407328161273 rpy=0 0 0
- joint right_steering_hinge_joint: origin xyz=0.10643 -0.1187 -0.10656 rpy=0 -0.061844 0 -> xyz=0.10643 -0.1087 -0.10656 rpy=0 -0.061844 0
